Commit message: Ajuste de inércia no URDF e implementação de filtros de velocidade linear e angular para melhorar a estabilidade (tambem foi abaixado o link do braço do robô)

File: src/prm_2026/description/robot.urdf.xacro (robot description, xacro)
@@ -59,5 +59,5 @@
       </geometry>
     </collision>
-    <xacro:box_inertia m="1" w="${base_width}" d="${base_length}" h="${base_height}"/>
+    <xacro:box_inertia m="0.2" w="${base_width}" d="${base_length}" h="${base_height}"/>
   </link>
   <!-- Definindo a Base do Robô (base footprint) -->
@@ -89,5 +89,5 @@
         </geometry>
       </collision>
-      <xacro:cylinder_inertia m="2.5" r="${wheel_radius}" h="${wheel_width}"/>
+      <xacro:cylinder_inertia m="0.2" r="${wheel_radius}" h="${wheel_width}"/>
     </link>
     <joint name="${prefix}_joint" type="continuous">
@@ -472,5 +472,5 @@
     <axis xyz="0 1 0"/>
     <limit effort="50.0" lower="-1.57075" upper="0.2" velocity="0.5"/>
-    <origin rpy="0 0 0" xyz="0.2 0 0.1"/>
+    <origin rpy="0 0 0" xyz="0.2 0 0.05"/>
     <parent link="base_link"/>
     <child link="gripper_pole"/>

Commit message: Change to NAV2, and start of visual SLAM

File: src/prm_2026/description/robot.urdf.xacro (robot description, xacro)
@@ -59,5 +59,5 @@
       </geometry>
     </collision>
-    <xacro:box_inertia m="0.2" w="${base_width}" d="${base_length}" h="${base_height}"/>
+    <xacro:box_inertia m="4.0" w="${base_width}" d="${base_length}" h="${base_height}"/>
   </link>
   <!-- Definindo a Base do Robô (base footprint) -->
@@ -89,5 +89,5 @@
         </geometry>
       </collision>
-      <xacro:cylinder_inertia m="0.2" r="${wheel_radius}" h="${wheel_width}"/>
+      <xacro:cylinder_inertia m="0.05" r="${wheel_radius}" h="${wheel_width}"/>
     </link>
     <joint name="${prefix}_joint" type="continuous">
@@ -101,4 +101,17 @@
   <xacro:wheel prefix="drivewhl_l" x_reflect="-1" y_reflect="1" />
   <xacro:wheel prefix="drivewhl_r" x_reflect="-1" y_reflect="-1" />
+  <!-- High friction on drive wheels (prevents slip) -->
+  <gazebo reference="drivewhl_l_link">
+    <mu1>100.0</mu1>
+    <mu2>50.0</mu2>
+    <kp>1e6</kp>
+    <kd>1.0</kd>
+  </gazebo>
+  <gazebo reference="drivewhl_r_link">
+    <mu1>100.0</mu1>
+    <mu2>50.0</mu2>
+    <kp>1e6</kp>
+    <kd>1.0</kd>
+  </gazebo>
   <link name="front_caster">
     <visual>
@@ -123,4 +136,11 @@
     <origin xyz="${caster_xoff} 0.0 ${-(base_height/2)}" rpy="0 0 0"/>
   </joint>
+  <!-- Very low friction on caster so it rotates freely -->
+  <gazebo reference="front_caster">
+    <mu1>0.01</mu1>
+    <mu2>0.01</mu2>
+    <kp>100000.0</kp>
+    <kd>1.0</kd>
+  </gazebo>
   <!-- Definindo a IMU do Robô (física) -->
   <link name="imu_link">
@@ -221,7 +241,7 @@
       <command_interface name="velocity">
         <!-- Valor mínimo permitido para o comando de velocidade (limite inferior) -->
-        <param name="min">-1</param>
+        <param name="min">-10</param>
         <!-- Valor máximo permitido para o comando de velocidade (limite superior) -->
-        <param name="max">1</param>
+        <param name="max">10</param>
       </command_interface>
       <!-- Interface de estado que fornece a posição atual da junta (por exemplo, em radianos) -->
@@ -235,7 +255,7 @@
       <command_interface name="velocity">
         <!-- Limite inferior da velocidade que pode ser comandada -->
-        <param name="min">-1</param>
+        <param name="min">-10</param>
         <!-- Limite superior da velocidade que pode ser comandada -->
-        <param name="max">1</param>
+        <param name="max">10</param>
       </command_interface>
       <!-- Interface de estado para leitura da posição da junta -->
@@ -383,4 +403,22 @@
       <enable_metrics>true</enable_metrics>
     </sensor> -->
+    <!-- RGB camera – used by bb8_visual_slam package (rtabmap loop closure) -->
+    <sensor name="robot_cam_rgb" type="camera">
+      <topic>robot_cam_rgb</topic>
+      <camera>
+        <horizontal_fov>1.57</horizontal_fov>
+        <image>
+          <width>320</width>
+          <height>240</height>
+        </image>
+        <clip>
+          <near>0.1</near>
+          <far>100</far>
+        </clip>
+      </camera>
+      <always_on>1</always_on>
+      <update_rate>10</update_rate>
+      <visualize>false</visualize>
+    </sensor>
     <!-- Insere uma camera com segmentacao semantica -->
     <sensor name="robot_cam" type="segmentation">
@@ -470,5 +508,5 @@
   </gazebo>
   <joint name="gripper_extension" type="revolute">
-    <axis xyz="0 1 0"/>
+    <axis xyz="0 0 1"/>
     <limit effort="50.0" lower="-1.57075" upper="0.2" velocity="0.5"/>
     <origin rpy="0 0 0" xyz="0.2 0 0.05"/>

Commit message: Navegação reativa

File: src/prm_2026/description/robot.urdf.xacro (robot description, xacro)
@@ -268,4 +268,12 @@
         <param name="min">-1.57075</param>
         <param name="max">0.2</param>
+      </command_interface>
+      <state_interface name="position"/>
+      <state_interface name="velocity"/>
+    </joint>
+    <joint name="arm_elbow">
+      <command_interface name="position">
+        <param name="min">-1.5708</param>
+        <param name="max">0.5</param>
       </command_interface>
       <state_interface name="position"/>
@@ -507,4 +515,5 @@
     </sensor> -->
   </gazebo>
+  <!-- Shoulder: sweeps arm sideways (Z-axis rotation) -->
   <joint name="gripper_extension" type="revolute">
     <axis xyz="0 0 1"/>
@@ -512,4 +521,28 @@
     <origin rpy="0 0 0" xyz="0.2 0 0.05"/>
     <parent link="base_link"/>
+    <child link="upper_arm"/>
+  </joint>
+  <!-- Upper arm segment (shoulder → elbow) -->
+  <link name="upper_arm">
+    <visual>
+      <geometry>
+        <cylinder length="0.15" radius="0.01"/>
+      </geometry>
+      <origin rpy="0 1.57075 0" xyz="0.075 0 0"/>
+    </visual>
+    <collision>
+      <geometry>
+        <cylinder length="0.15" radius="0.01"/>
+      </geometry>
+      <origin rpy="0 1.57075 0" xyz="0.075 0 0"/>
+    </collision>
+    <xacro:cylinder_inertia m="0.005" r="0.01" h="0.15"/>
+  </link>
+  <!-- Elbow: folds lower arm back toward body (same Z-axis rotation) -->
+  <joint name="arm_elbow" type="revolute">
+    <axis xyz="0 0 1"/>
+    <limit effort="50.0" lower="-1.5708" upper="0.5" velocity="0.5"/>
+    <origin xyz="0.15 0 0" rpy="0 0 0"/>
+    <parent link="upper_arm"/>
     <child link="gripper_pole"/>
   </joint>
